File: Electrical/modules/pcb/board.brd (EAGLE design)
At the start: 127 x 127 mm, 21 parts, among them IC1 OP-AMP, IC2 LM311N, U1 UA7805CKCS, U2 UA7805CKCS

Commit message: pcb
Parts:
- removed C3: 0.1uF, SparkFun-Capacitors:CAP-PTH-SMALL-KIT
- removed C4: 0.33uF, SparkFun-Capacitors:CAP-PTH-SMALL-KIT
- removed J1: (no value), SparkFun-Connectors:1X02
- removed U2: UA7805CKCS, regulator:KCS3
- added C10, C13, C14, C15, C16, C17, C18, C8: 0.1uF, SparkFun-Capacitors:CAP-PTH-SMALL-KIT
- added C11, C9: 100nf, Seeed-Capacitor:CERAMIC-2.54
- added C12, C19: 1uF, SparkFun-Capacitors:CAP-PTH-SMALL-KIT
- added J4, J6: (no value), SparkFun-Connectors:1X02
- added Q1, Q2, Q5, Q6: IRF3505, IRF3505:TO-220AB
- added R17, R18, R22, R24, R37, R38, R42, R44: 10k, SparkFun-Resistors:AXIAL-0.3
- added R19, R21, R23, R26, R39, R41, R43, R46: 100, SparkFun-Resistors:AXIAL-0.3
- added R20, R25, R40, R45: 33k, SparkFun-Resistors:AXIAL-0.3
- added T13, T14, T5, T6: 2N3904, transistor:TO92
- added T15, T16, T7, T8: 2N3906BU, 2N3906:TO-92
- added U10, U5, U6, U9: HUF75321, HUF75321:TO-220
- moved C5 96.9 mm to (16.5, 7.62), turned to 90 degrees
- moved R1 96.6 mm to (19.1, 16.5), turned to 0 degrees
- moved IC2 90.4 mm to (8.89, 7.62), turned to 180 degrees
- moved QSD1 81.0 mm to (6.35, 43.2), turned to 90 degrees
- moved C7 78.8 mm to (16.5, 25.4)
- moved IC1 78.8 mm to (8.89, 24.1)
- moved R2 78.8 mm to (8.89, 15.2)
- moved R6 78.8 mm to (8.89, 33.0)
- moved R3 78.8 mm to (8.89, 30.5)
- moved R4 78.8 mm to (8.89, 17.8)
- moved R5 78.8 mm to (8.89, 35.6)
- moved C6 65.8 mm to (14.0, 43.2), turned to 90 degrees
- moved C2 11.5 mm to (63.5, 104.1)
- moved J2 11.5 mm to (64.8, 109.2)
- moved U1 11.5 mm to (64.8, 99.1)
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Connections:
- removed net 5V_IC: C1.1, C5.1, C6.1, C7.1, IC1.8, IC2.8, QSD1.+, R1.3, R4.P$2, R6.P$2, U1.1
- removed net 5V_STM: C3.1, U$1.E5V, U2.1
- removed net V_IN: C4.1, J1.2, U2.3
- new net 5V_SUPPLY: C1.1, C5.1, C6.1, C7.1, IC1.8, IC2.8, QSD1.+, R1.3, R4.P$2, R6.P$2, U$1.E5V, U1.1
- new net LEFT_1: T13.2
- new net LEFT_2: T14.2
- new net N$17: Q1.1, R18.P$1, R19.P$2, R25.P$2
- new net N$18: R19.P$1, T5.1
- new net N$19: R23.P$1, T6.1
- new net N$20: R17.P$2, R21.P$1, U6.1
- new net N$21: R21.P$2, T7.3
- new net N$22: R20.P$2, T7.2
- new net N$23: R24.P$2, R26.P$1, U5.1
- new net N$24: R26.P$2, T8.3
- new net N$25: R25.P$1, T8.2
- new net N$26: Q2.1, R20.P$1, R22.P$1, R23.P$2
- new net N$27: C9.2, J4.1, Q2.2, U5.2
- new net N$41: Q5.1, R38.P$1, R39.P$2, R45.P$2
- new net N$42: R39.P$1, T13.1
- new net N$43: R43.P$1, T14.1
- new net N$44: R37.P$2, R41.P$1, U10.1
- new net N$45: R41.P$2, T15.3
- new net N$46: R40.P$2, T15.2
- new net N$47: R44.P$2, R46.P$1, U9.1
- new net N$48: R46.P$2, T16.3
- new net N$49: R45.P$1, T16.2
- new net N$50: Q6.1, R40.P$1, R42.P$1, R43.P$2
- new net N$51: C11.2, J6.1, Q6.2, U9.2
- new net N$8: C9.1, J4.2, Q1.2, U6.2
- new net N$9: C11.1, J6.2, Q5.2, U10.2
- new net RIGHT_1: T5.2
- new net RIGHT_2: T6.2
- new net VCC: C10.1, C12.1, C13.1, C14.1, C15.1, C16.1, C17.1, C18.1, C19.1, C8.1, Q1.3, Q2.3, Q5.3, Q6.3, R18.P$2, R22.P$2, R38.P$2, R42.P$2, T15.1, T16.1, T7.1, T8.1
- net GND: now also C10.2, C12.2, C13.2, C14.2, C15.2, C16.2, C17.2, C18.2, C19.2, C8.2, R17.P$1, R24.P$1, R37.P$1, R44.P$1, T13.3, T14.3, T5.3, T6.3, U10.3, U5.3, U6.3, U9.3; no longer C3.2, C4.2, J1.1, U2.2
Routing:
- net N$6: track 0.00 -> 127.0 mm
Other:
- board text added: "5V Reg"
- board text added: "H_Bridges"
- board text added: "IR Sensor"

Commit message: circuit updates
Parts:
- removed R2: 20k, SparkFun-Resistors:AXIAL-0.3
- added C20: 0.33uF, SparkFun-Capacitors:CAP-PTH-SMALL-KIT
- added C21, C23, C4: 0.1uF, SparkFun-Capacitors:CAP-PTH-SMALL-KIT
- added C22, C24: 1uF, SparkFun-Capacitors:CAP-PTH-SMALL-KIT
- added C3: 470pF, SparkFun-Capacitors:CAP-PTH-SMALL-KIT
- added D1, D2: 1N4004, adafruit:DO41-10
- added IC4, IC5: LM311N, linear:DIL08
- added J1: (no value), SparkFun-Connectors:DEANS
- added R10: (no value), resistor:RTRIMT93YA
- added R13, R15, R16, R28: 47k, rcl:0204/5
- added R14, R27: 300, rcl:0204/5
- added R7, R8, R9: 10k, SparkFun-Resistors:AXIAL-0.3
- added U2: UA7805CKCS, regulator:KCS3
- added U3, U4: QRD1114, SparkFun-Sensors:QRD1114
- added VR2, VR3: 5k, SparkFun-Resistors:TRIMPOT-SMD-5MM
- R3: value 20k -> 33k
- moved R6 88.4 mm to (83.8, 80.0)
- moved R3 16.1 mm to (24.1, 25.4)
Connections:
- net VCC renamed LIPO_SUPPLY
- removed net 5V_SUPPLY: C1.1, C5.1, C6.1, C7.1, IC1.8, IC2.8, QSD1.+, R1.3, R4.P$2, R6.P$2, U$1.E5V, U1.1
- removed net N$5: IC1.6, R2.P$1, R4.P$1
- new net 5V_AC: C1.1, C21.1, C22.1, C23.1, C24.1, C5.1, C6.1, C7.1, D1.A, IC1.8, IC2.8, IC4.5, IC5.5, QSD1.+, R1.3, R13.2, R14.2, R15.2, R16.2, R27.2, R28.2, U1.1, VR2.A, VR3.A
- new net 5V_DC: C4.1, D2.A, U$1.E5V, U2.1
- new net N$10: R9.P$2, T14.2
- new net N$11: R8.P$1, T13.2
- new net N$14: R7.P$2, T6.2
- new net N$15: R6.P$1, T5.2
- new net N$16: R14.1, U3.3
- new net N$28: IC4.3, R13.1, U3.1
- new net N$29: IC4.2, VR2.B
- new net N$30: R27.1, U4.3
- new net N$31: IC5.3, R16.1, U4.1
- new net N$32: IC5.2, VR3.B
- new net N$7: IC1.1, IC1.2, R3.P$1
- new net V+: IC4.8, IC5.8
- new net VOUT: IC4.7, IC5.7, R15.1, R28.1
- new net V_IN2: C20.1, D2.C, J1.+, U2.3
- net GND: now also C20.2, C21.2, C22.2, C23.2, C24.2, C3.2, C4.2, IC4.1, IC4.4, IC5.1, IC5.4, J1.-, R4.P$2, U2.2, U3.2, U3.4, U4.2, U4.4, VR2.C, VR3.C
- net LEFT_1: now also R8.P$2; no longer T13.2
- net LEFT_2: now also R9.P$1; no longer T14.2
- net N$2: now also C3.1; no longer IC1.1
- net N$3: now also R10.2; no longer R2.P$2
- net N$4: now also IC1.6, R10.3, R4.P$1; no longer IC1.2, R3.P$1, R6.P$1
- net RIGHT_1: now also R6.P$2; no longer T5.2
- net RIGHT_2: now also R7.P$1; no longer T6.2
- net V_IN1: now also D1.C

Commit message: updates
Parts:
- removed C10, C13, C14, C15, C16, C17, C18, C8: 0.1uF, SparkFun-Capacitors:CAP-PTH-SMALL-KIT
- removed C11, C9: 100nf, Seeed-Capacitor:CERAMIC-2.54
- removed C12, C19: 1uF, SparkFun-Capacitors:CAP-PTH-SMALL-KIT
- removed D2: 1N4004, adafruit:DO41-10
- removed IC2: LM311N, linear:DIL08
- removed J1: (no value), SparkFun-Connectors:DEANS
- removed J2, J4, J6: (no value), SparkFun-Connectors:1X02
- removed Q1, Q2, Q5, Q6: IRF3505, IRF3505:TO-220AB
- removed R17, R18, R22, R24, R37, R38, R42, R44, R6, R7, R8, R9: 10k, SparkFun-Resistors:AXIAL-0.3
- removed R19, R21, R23, R26, R39, R41, R43, R46: 100, SparkFun-Resistors:AXIAL-0.3
- removed R20, R25, R40, R45: 33k, SparkFun-Resistors:AXIAL-0.3
- removed T13, T14, T5, T6: 2N3904, transistor:TO92
- removed T15, T16, T7, T8: 2N3906BU, 2N3906:TO-92
- removed U1, U2: UA7805CKCS, regulator:KCS3
- removed U10, U5, U6, U9: HUF75321, HUF75321:TO-220
- added LIPO_B: (no value), SparkFun-Connectors:DEANS
- added LIPO_SMALL_1, LIPO_SMALL_2: (no value), SparkFun-Connectors:1X02
- added QSD2: (no value), Seeed-LED:LED2-2.54-D5.0MM
- added R2: 10k, SparkFun-Resistors:AXIAL-0.3
- added U$2, U$3: DC-DC-STEP-DOWN-LM2596, diy-modules:DC-DC-STEP-DOWN-LM2596
- added U$4: UA7805, TO220:TO-220AB
- C20: value 0.33uF -> 1U; device SparkFun-Capacitors:CAP-PTH-SMALL-KIT -> capacitor-wima:C5B5
- C3: value 470pF -> 1U; device SparkFun-Capacitors:CAP-PTH-SMALL-KIT -> capacitor-wima:C5B5
- C4, C7: value 0.1uF -> 1U; device SparkFun-Capacitors:CAP-PTH-SMALL-KIT -> capacitor-wima:C5B5
- R1: value (none) -> 1k; device resistor:RTRIMT93YA -> SparkFun-Resistors:AXIAL-0.3
- R10: value (none) -> 100k
- R3: value 33k -> 100k; device SparkFun-Resistors:AXIAL-0.3 -> resistor:RTRIMT93YA
- moved C7 407.7 mm to (-30.1, -379.6), turned to 0 degrees
- moved C20 377.8 mm to (-30.1, -395.6)
- moved C3 359.1 mm to (-30.1, -347.6)
- moved C4 342.8 mm to (-30.1, -363.6)
- moved R3 196.8 mm to (-34.3, -162.6)
- moved R1 141.4 mm to (-2.54, -123.2)
Connections:
- removed net 5V_AC: C1.1, C21.1, C22.1, C23.1, C24.1, C5.1, C6.1, C7.1, D1.A, IC1.8, IC2.8, IC4.5, IC5.5, QSD1.+, R1.3, R13.2, R14.2, R15.2, R16.2, R27.2, R28.2, U1.1, VR2.A, VR3.A
- removed net GPIO_IR: IC2.7
- removed net LEFT_1: R8.P$2
- removed net LEFT_2: R9.P$1
- removed net LIPO_SUPPLY: C10.1, C12.1, C13.1, C14.1, C15.1, C16.1, C17.1, C18.1, C19.1, C8.1, Q1.3, Q2.3, Q5.3, Q6.3, R18.P$2, R22.P$2, R38.P$2, R42.P$2, T15.1, T16.1, T7.1, T8.1
- removed net N$10: R9.P$2, T14.2
- removed net N$11: R8.P$1, T13.2
- removed net N$14: R7.P$2, T6.2
- removed net N$15: R6.P$1, T5.2
- removed net N$17: Q1.1, R18.P$1, R19.P$2, R25.P$2
- removed net N$18: R19.P$1, T5.1
- removed net N$19: R23.P$1, T6.1
- removed net N$20: R17.P$2, R21.P$1, U6.1
- removed net N$21: R21.P$2, T7.3
- removed net N$22: R20.P$2, T7.2
- removed net N$23: R24.P$2, R26.P$1, U5.1
- removed net N$24: R26.P$2, T8.3
- removed net N$25: R25.P$1, T8.2
- removed net N$26: Q2.1, R20.P$1, R22.P$1, R23.P$2
- removed net N$27: C9.2, J4.1, Q2.2, U5.2
- removed net N$41: Q5.1, R38.P$1, R39.P$2, R45.P$2
- removed net N$42: R39.P$1, T13.1
- removed net N$43: R43.P$1, T14.1
- removed net N$44: R37.P$2, R41.P$1, U10.1
- removed net N$45: R41.P$2, T15.3
- removed net N$46: R40.P$2, T15.2
- removed net N$47: R44.P$2, R46.P$1, U9.1
- removed net N$48: R46.P$2, T16.3
- removed net N$49: R45.P$1, T16.2
- removed net N$50: Q6.1, R40.P$1, R42.P$1, R43.P$2
- removed net N$51: C11.2, J6.1, Q6.2, U9.2
- removed net N$7: IC1.1, IC1.2, R3.P$1
- removed net N$8: C9.1, J4.2, Q1.2, U6.2
- removed net N$9: C11.1, J6.2, Q5.2, U10.2
- removed net RIGHT_1: R6.P$2
- removed net RIGHT_2: R7.P$1
- removed net V_IN2: C20.1, D2.C, J1.+, U2.3
- new net 5V_ANOLOG: C1.1, C21.1, C22.1, C23.1, C24.1, C5.1, C6.1, D1.A, IC1.8, IC4.5, IC5.5, QSD1.+, QSD2.+, R13.2, R14.2, R15.2, R16.2, R27.2, R28.2, U$4.3, VR2.A, VR3.A
- new net 5V_DIGITAL: C20.1, C3.1, C4.1, C7.1, U$3.OUT+
- new net 6V_SERVO: U$2.OUT+
- new net IR_1: IC1.7, R10.2
- new net IR_3: IC1.1, R3.2
- new net LIPO_B_GND: LIPO_B.-, U$3.IN-
- new net LIPO_B_SUPPLY: LIPO_B.+, U$3.IN+
- new net OUTPUT2: IC1.3, QSD2.-, R1.P$2
- net 5V_DC: no longer C4.1, D2.A, U2.1
- net GND: now also LIPO_SMALL_1.1, R1.P$1, R2.P$2, U$2.OUT-, U$3.OUT-, U$4.2; no longer C10.2, C12.2, C13.2, C14.2, C15.2, C16.2, C17.2, C18.2, C19.2, C8.2, IC2.1, IC2.4, J1.-, J2.1, R1.1, R17.P$1, R24.P$1, R37.P$1, R44.P$1, T13.3, T14.3, T5.3, T6.3, U1.2, U10.3, U2.2, U5.3, U6.3, U9.3
- net N$1: now also LIPO_SMALL_2.2, U$2.IN+; no longer IC2.2, R1.2
- net N$2: now also IC1.2, R2.P$1, R3.3; no longer C3.1, IC1.5, R3.P$2
- net N$3: now also LIPO_SMALL_2.1, U$2.IN-; no longer IC1.7, IC2.3, R10.2
- net OUTPUT1: now also IC1.5; no longer IC1.3
- net V_IN1: now also LIPO_SMALL_1.2, U$4.1; no longer J2.2, U1.3

Commit message: updates
Parts:
- added M1, M2, M3: SERVO, SparkFun-Electromechanical:1X03
- added R11, R12, R9: 1k, SparkFun-Resistors:AXIAL-0.3
- added U$5: ENCODER, TO220:TO-220AB
- added U$6: RPI3, Raspberry_Pi_3:PI
Connections:
- net IR_3 renamed IR_2
- removed net 5V_DC: U$1.E5V
- new net +5V: R11.P$2, R12.P$2, R9.P$2, U$1.+5V
- new net ENCODER_1: U$5.1
- new net ENCODER_2: U$5.2
- new net SERVO_BASKET: M3.1
- new net SERVO_CLAW_1: M2.1
- new net SERVO_CLAW_2: M1.1
- net 5V_DIGITAL: now also U$1.E5V
- net 6V_SERVO: now also M1.2, M2.2, M3.2, R11.P$1, R12.P$1, R9.P$1
- net GND: now also M1.3, M2.3, M3.3, U$5.3
Changed lines of the file:
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@@
 <element name="C20" library="capacitor-wima" library_urn="urn:adsk.eagle:library:116" package="C5B5" package3d_urn="urn:adsk.eagle:package:5428/1" value="1U" x="-30.099" y="-395.605"/>
 <element name="U$4" library="TO220" package="TO-220AB" value="UA7805" x="-26.6065" y="-412.5595"/>
+<element name="M1" library="SparkFun-Electromechanical" library_urn="urn:adsk.eagle:library:516" package="1X03" package3d_urn="urn:adsk.eagle:package:38562/1" value="SERVO" x="-31.242" y="-430.911"/>
+<element name="M2" library="SparkFun-Electromechanical" library_urn="urn:adsk.eagle:library:516" package="1X03" package3d_urn="urn:adsk.eagle:package:38562/1" value="SERVO" x="-31.242" y="-449.707"/>
+<element name="M3" library="SparkFun-Electromechanical" library_urn="urn:adsk.eagle:library:516" package="1X03" package3d_urn="urn:adsk.eagle:package:38562/1" value="SERVO" x="-31.242" y="-468.503"/>
+<element name="R9" library="SparkFun-Resistors" library_urn="urn:adsk.eagle:library:532" package="AXIAL-0.3" package3d_urn="urn:adsk.eagle:package:39658/1" value="1k" x="-27.432" y="-543.687">
+<attribute name="PROD_ID" value="RES-08380" x="-27.432" y="-543.687" size="1.778" layer="27" display="off"/>
+</element>
+<element name="R11" library="SparkFun-Resistors" library_urn="urn:adsk.eagle:library:532" package="AXIAL-0.3" package3d_urn="urn:adsk.eagle:package:39658/1" value="1k" x="-27.432" y="-562.483">
+<attribute name="PROD_ID" value="RES-08380" x="-27.432" y="-562.483" size="1.778" layer="27" display="off"/>
+</element>
+<element name="R12" library="SparkFun-Resistors" library_urn="urn:adsk.eagle:library:532" package="AXIAL-0.3" package3d_urn="urn:adsk.eagle:package:39658/1" value="1k" x="-27.432" y="-581.279">
+<attribute name="PROD_ID" value="RES-08380" x="-27.432" y="-581.279" size="1.778" layer="27" display="off"/>
+</element>
+<element name="U$5" library="TO220" package="TO-220AB" value="ENCODER" x="-26.6065" y="-599.6305"/>
+<element name="U$6" library="Raspberry_Pi_3" package="PI" value="RPI3" x="-39.624" y="-671.7538"/>
 </elements>
 <signals>
@@
 <contactref element="U$4" pad="2"/>
 <contactref element="LIPO_SMALL_1" pad="1"/>
+<contactref element="M3" pad="3"/>
+<contactref element="M2" pad="3"/>
+<contactref element="M1" pad="3"/>
+<contactref element="U$5" pad="3"/>
 <wire x1="156.02" y1="76.2" x2="163.64" y2="76.2" width="0" layer="19" extent="1-1"/>
 <wire x1="161.1" y1="68.58" x2="163.64" y2="76.2" width="0" layer="19" extent="1-1"/>
@@
 <wire x1="-27.559" y1="-395.605" x2="-27.559" y2="-379.603" width="0" layer="19" extent="1-1"/>
 <wire x1="-29.1465" y1="-412.5595" x2="-27.559" y2="-395.605" width="0" layer="19" extent="1-1"/>
+<wire x1="-26.162" y1="-430.911" x2="-29.1465" y2="-412.5595" width="0" layer="19" extent="1-1"/>
+<wire x1="-26.162" y1="-449.707" x2="-26.162" y2="-430.911" width="0" layer="19" extent="1-1"/>
+<wire x1="-26.162" y1="-468.503" x2="-26.162" y2="-449.707" width="0" layer="19" extent="1-1"/>
+<wire x1="-26.6065" y1="-599.6305" x2="-26.162" y2="-468.503" width="0" layer="19" extent="1-1"/>
 </signal>
 <signal name="V_IN1">
@@
 <contactref element="VR3" pad="B"/>
 <wire x1="179.07" y1="84.5185" x2="156.02" y2="68.58" width="0" layer="19" extent="1-1"/>
-</signal>
-<signal name="5V_DC">
-<contactref element="U$1" pad="E5V"/>
 </signal>
 <signal name="5V_ANOLOG">
@@
 <wire x1="7.62" y1="27.94" x2="1.27" y2="-123.19" width="0" layer="19" extent="1-1"/>
 </signal>
-<signal name="IR_3">
+<signal name="IR_2">
 <contactref element="R3" pad="2"/>
 <contactref element="IC1" pad="1"/>
@@
 <signal name="6V_SERVO">
 <contactref element="U$2" pad="OUT+"/>
+<contactref element="M3" pad="2"/>
+<contactref element="M2" pad="2"/>
+<contactref element="M1" pad="2"/>
+<contactref element="R12" pad="P$1"/>
+<contactref element="R11" pad="P$1"/>
+<contactref element="R9" pad="P$1"/>
+<wire x1="-28.702" y1="-449.707" x2="-28.702" y2="-468.503" width="0" layer="19" extent="1-1"/>
+<wire x1="-28.702" y1="-430.911" x2="-28.702" y2="-449.707" width="0" layer="19" extent="1-1"/>
+<wire x1="-31.242" y1="-543.687" x2="-28.702" y2="-468.503" width="0" layer="19" extent="1-1"/>
+<wire x1="-31.242" y1="-562.483" x2="-31.242" y2="-543.687" width="0" layer="19" extent="1-1"/>
+<wire x1="-31.242" y1="-581.279" x2="-31.242" y2="-562.483" width="0" layer="19" extent="1-1"/>
+<wire x1="12.192" y1="-184.404" x2="-28.702" y2="-430.911" width="0" layer="19" extent="1-1"/>
 </signal>
 <signal name="LIPO_B_SUPPLY">
@@
 <contactref element="C7" pad="1"/>
 <contactref element="C20" pad="1"/>
+<contactref element="U$1" pad="E5V"/>
 <wire x1="-32.639" y1="-379.603" x2="-32.639" y2="-395.605" width="0" layer="19" extent="1-1"/>
 <wire x1="-32.639" y1="-363.601" x2="-32.639" y2="-379.603" width="0" layer="19" extent="1-1"/>
 <wire x1="-32.639" y1="-347.599" x2="-32.639" y2="-363.601" width="0" layer="19" extent="1-1"/>
 <wire x1="12.192" y1="-270.764" x2="-32.639" y2="-347.599" width="0" layer="19" extent="1-1"/>
+<wire x1="35.56" y1="44.45" x2="12.192" y2="-270.764" width="0" layer="19" extent="1-1"/>
+</signal>
+<signal name="SERVO_CLAW_2">
+<contactref element="M1" pad="1"/>
+</signal>
+<signal name="SERVO_CLAW_1">
+<contactref element="M2" pad="1"/>
+</signal>
+<signal name="SERVO_BASKET">
+<contactref element="M3" pad="1"/>
+</signal>
+<signal name="+5V">
+<contactref element="R9" pad="P$2"/>
+<contactref element="R11" pad="P$2"/>
+<contactref element="R12" pad="P$2"/>
+<contactref element="U$1" pad="+5V"/>
+<wire x1="-23.622" y1="-562.483" x2="-23.622" y2="-581.279" width="0" layer="19" extent="1-1"/>
+<wire x1="-23.622" y1="-543.687" x2="-23.622" y2="-562.483" width="0" layer="19" extent="1-1"/>
+<wire x1="35.56" y1="29.21" x2="-23.622" y2="-543.687" width="0" layer="19" extent="1-1"/>
+</signal>
+<signal name="ENCODER_1">
+<contactref element="U$5" pad="1"/>
+</signal>
+<signal name="ENCODER_2">
+<contactref element="U$5" pad="2"/>
 </signal>
 </signals>

Commit message: updates
Parts:
- removed VR2, VR3: 5k, SparkFun-Resistors:TRIMPOT-SMD-5MM
- added C13, C15, C18, C25: 1uF, SparkFun-Capacitors:CAP-PTH-SMALL-KIT
- added C14, C16, C17, C19, C26, C27: 0.1uF, SparkFun-Capacitors:CAP-PTH-SMALL-KIT
- added D4, D5, D6, D7: 15V, diode:DO41Z10
- added J2, J3: (no value), SparkFun-Connectors:1X02
- added R17, R18, R19, R20, R21, R22, R23, R24, R25, R26, R29, R30, R31, R6, R7, R8: 1k, SparkFun-Resistors:AXIAL-0.3
- added R32, R33: 10k, resistor:RTRIMT93YA
- added U$11, U$12, U$13, U$14, U$15, U$16, U$17, U$18: HUF75321, TO220:TO-220AB
- added U2, U5: LT1161CNPBF, LT1161NC:PDIP-20_N
- R13, R15, R16, R28: value 47k -> 1k; device rcl:0204/5 -> SparkFun-Resistors:AXIAL-0.3
- R14, R27: value 300 -> 1k; device rcl:0204/5 -> SparkFun-Resistors:AXIAL-0.3
- moved U$6 717.3 mm to (57.0, 39.0), turned to 90 degrees
- moved U$5 637.5 mm to (6.00, 37.0), turned to 180 degrees
- moved R12 634.6 mm to (37.0, 50.0)
- moved R11 620.8 mm to (37.0, 55.0)
- moved R9 610.0 mm to (36.0, 63.0)
- moved M3 588.9 mm to (79.0, 110.0)
- moved M2 568.8 mm to (70.0, 110.0)
- moved M1 548.6 mm to (60.0, 110.0)
- moved C20 513.1 mm to (20.0, 115.0), turned to 270 degrees
- moved C7 508.0 mm to (72.0, 118.0), turned to 270 degrees
- moved C4 482.0 mm to (27.0, 115.0), turned to 270 degrees
- moved C3 475.0 mm to (64.0, 118.0), turned to 270 degrees
- moved U$4 425.9 mm to (62.0, 4.00)
- moved U$3 418.4 mm to (42.0, 136.0), turned to 270 degrees
- moved LIPO_B 381.1 mm to (58.0, 140.0), turned to 180 degrees
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Connections:
- removed net N$32: IC5.2, VR3.B
- new net HB_LEFT_1: U5.3, U5.7
- new net HB_LEFT_2: U5.5, U5.9
- new net HB_RIGHT_1: U2.3, U2.7
- new net HB_RIGHT_2: U2.5, U2.9
- new net N$10: R17.P$1, R26.P$1, R29.P$2
- new net N$11: R29.P$1, R30.P$2, R8.P$1
- new net N$12: R30.P$1, R31.P$2, R7.P$1
- new net N$20: U$11.1, U2.18
- new net N$21: U$12.1, U2.16
- new net N$22: D5.C, U$14.1, U2.14
- new net N$23: D4.C, U$13.1, U2.12
- new net N$24: C17.2, J2.1, U$12.3, U$14.2
- new net N$25: C17.1, J2.2, U$11.3, U$13.2
- new net N$26: U$15.1, U5.18
- new net N$27: U$16.1, U5.16
- new net N$33: D7.C, U$18.1, U5.14
- new net N$34: D6.C, U$17.1, U5.12
- new net N$35: C27.2, J3.1, U$16.3, U$18.2
- new net N$36: C27.1, J3.2, U$15.3, U$17.2
- new net N$5: R21.P$1, R22.P$1, R23.P$2
- new net N$6: IC5.2, R32.2
- new net N$7: R20.P$1, R23.P$1, R24.P$2
- new net N$8: R19.P$1, R24.P$1, R25.P$2
- new net N$9: R18.P$1, R25.P$1, R26.P$2
- new net PI_INT: U$6.4
- new net PI_RX: U$6.31
- new net PI_TX: U$6.33
- new net R1: R21.P$2, U$6.19
- new net R2: R20.P$2, U$6.23
- new net R3: R19.P$2, U$6.25
- new net R4: R18.P$2, U$6.26
- new net R5: R17.P$2, U$6.28
- new net R6: R8.P$2, U$6.30
- new net R7: R7.P$2, U$6.29
- new net R8: R6.P$2, U$6.34
- new net RPI_ANALOG: R31.P$1, R6.P$1
- new net VCC: C18.1, C19.1, C25.1, C26.1, U$15.2, U$16.2, U5.11, U5.13, U5.15, U5.17, U5.19, U5.20
- net 5V_ANOLOG: now also R13.P$2, R14.P$2, R15.P$2, R16.P$2, R27.P$2, R28.P$2, R32.3, R33.3; no longer R13.2, R14.2, R15.2, R16.2, R27.2, R28.2, VR2.A, VR3.A
- net 5V_DIGITAL: now also U$6.37, U$6.39
- net GND: now also C15.2, C16.2, C18.2, C19.2, C25.2, C26.2, D6.A, D7.A, R22.P$2, R32.1, R33.1, U$17.3, U$18.3, U$6.11, U$6.16, U$6.2, U$6.21, U$6.27, U$6.32, U$6.35, U$6.7, U5.1, U5.10; no longer VR2.C, VR3.C
- net LIPO_B_GND: now also C13.2, C14.2, D4.A, D5.A, U$13.3, U$14.3, U2.1, U2.10
- net LIPO_B_SUPPLY: now also C13.1, C14.1, C15.1, C16.1, U$11.2, U$12.2, U2.11, U2.13, U2.15, U2.17, U2.19, U2.20
- net N$16: now also R14.P$1; no longer R14.1
- net N$28: now also R13.P$1; no longer R13.1
- net N$29: now also R33.2; no longer VR2.B
- net N$30: now also R27.P$1; no longer R27.1
- net N$31: now also R16.P$1; no longer R16.1
- net VOUT: now also R15.P$1, R28.P$1; no longer R15.1, R28.1
Routing:
- net N$6: track 127.0 -> 0.00 mm
- removed copper zone on layer 1, net GND
Other:
- board size 127 x 127 mm -> 88.9 x 158.8 mm
- board text removed: "5V Reg"
- board text removed: "H_Bridges"
- board text removed: "IR Sensor"

Commit message: updates
Parts:
- moved LIPO_SMALL_2 87.7 mm to (73.5, 112.5), turned to 180 degrees
- moved M1 85.6 mm to (54.6, 24.5)
- moved M2 85.6 mm to (64.6, 24.5)
- moved M3 85.6 mm to (74.8, 24.5)
- moved R12 56.4 mm to (86.1, 22.2), turned to 270 degrees
- moved R11 54.0 mm to (78.9, 20.9), turned to 180 degrees
- moved R9 52.0 mm to (66.6, 20.9), turned to 180 degrees
- moved J2 46.4 mm to (41.5, 136.5), turned to 90 degrees
- moved C17 39.7 mm to (46.5, 137.5), turned to 270 degrees
- moved C27 39.6 mm to (44.0, 128.0), turned to 270 degrees
- moved C23 38.5 mm to (34.4, 22.8), turned to 90 degrees
- moved J3 38.0 mm to (49.5, 127.0), turned to 90 degrees
- moved U$17 37.9 mm to (37.0, 122.7), turned to 0 degrees
- moved U$15 37.7 mm to (34.2, 151.9), turned to 0 degrees
- moved U$13 37.1 mm to (52.0, 153.0), turned to 180 degrees
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Connections:
- removed net LIPO_B_GND: C13.2, C14.2, D4.A, D5.A, LIPO_B.-, U$13.3, U$14.3, U$3.IN-, U2.1, U2.10
- removed net N$3: LIPO_SMALL_2.1, U$2.IN-
- removed net VCC: C18.1, C19.1, C25.1, C26.1, U$15.2, U$16.2, U5.11, U5.13, U5.15, U5.17, U5.19, U5.20
- net 6V_SERVO: no longer R11.P$1, R12.P$1, R9.P$1
- net GND: now also C13.2, C14.2, D4.A, D5.A, LIPO_B.-, LIPO_SMALL_2.1, U$13.3, U$14.3, U$2.IN-, U$3.IN-, U2.1, U2.10
- net LIPO_B_SUPPLY: now also C18.1, C19.1, C25.1, C26.1, U$15.2, U$16.2, U5.11, U5.13, U5.15, U5.17, U5.19, U5.20
- net SERVO_BASKET: now also R12.P$1
- net SERVO_CLAW_1: now also R11.P$1
- net SERVO_CLAW_2: now also R9.P$1
Routing:
- net 5V_DIGITAL: track 0.00 -> 110.0 mm
- net N$36: track 0.00 -> 44.4 mm
- net N$25: track 0.00 -> 44.3 mm
- net N$35: track 0.00 -> 42.7 mm
- net 6V_SERVO: track 0.00 -> 40.3 mm
- net N$24: track 0.00 -> 32.1 mm
- net LIPO_B_SUPPLY: track 0.00 -> 31.4 mm
- net GND: track 0.00 -> 30.6 mm
- net N$23: track 0.00 -> 25.9 mm
- net N$22: track 0.00 -> 23.2 mm
- net N$34: track 0.00 -> 21.0 mm
- net N$26: track 0.00 -> 20.1 mm
- net N$1: track 0.00 -> 18.7 mm
- net N$20: track 0.00 -> 18.3 mm
- net N$9: track 0.00 -> 17.5 mm
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- added copper zone on layer 16, net GND
- added copper zone on layer 1, net LIPO_B_SUPPLY

Commit message: almost there
Parts:
- R17, R18, R19, R20, R21, R22, R6, R7, R8: value 1k -> 100k
- R23, R24, R25, R26, R29, R30, R31: value 1k -> 50k
- moved U$5 26.5 mm to (13.6, 57.4), turned to 270 degrees
