File: Electrical/modules/pcb/board.brd (EAGLE design)
At the start: 88.9 x 158.8 mm, 91 parts, among them IC1 OP-AMP, IC4 LM311N, IC5 LM311N, M1 SERVO, M2 SERVO, M3 SERVO, U2 LT1161CNPBF, U3 QRD1114, U4 QRD1114, U5 LT1161CNPBF

Commit message: updates
Parts:
- added C10, C12, C8: 0.1uF, SparkFun-Capacitors:CAP-PTH-SMALL-KIT
- added C11, C28, C9: 1uF, SparkFun-Capacitors:CAP-PTH-SMALL-KIT
- added IC2, IC3, IC6: LM311N, linear:DIL08
- added R34: 47k, SparkFun-Resistors:AXIAL-0.3
- added R35, R37, R38: 10k, resistor:RTRIMT93YA
- added R36: 300, SparkFun-Resistors:AXIAL-0.3
- added U$7: ENCODER, TO220:TO-220AB
- added U1, U6: QRD1114, SparkFun-Sensors:QRD1114
- R13, R15, R16: value 1k -> 47k
- R14, R27, R28: value 1k -> 300
- moved LIPO_SMALL_1 25.5 mm to (29.9, 13.9), turned to 90 degrees
- moved R28 20.0 mm to (52.3, 19.6), flipped to the bottom, turned to 90 degrees
- moved C2 19.2 mm to (34.9, 11.1), turned to 180 degrees
- moved M1 12.5 mm to (67.0, 25.8), turned to 270 degrees
- moved R15 10.9 mm to (46.2, 22.1), flipped to the bottom
- moved C1 10.8 mm to (65.1, 4.11), turned to 270 degrees
- moved C24 10.3 mm to (34.6, 5.35)
- moved R32 9.08 mm to (73.6, 3.75), turned to 90 degrees
- moved R14 7.73 mm to (57.6, 12.7)
- moved M2 7.22 mm to (71.7, 25.8), turned to 270 degrees
- moved R33 6.10 mm to (28.9, 6.25)
- moved QSD1 5.71 mm to (22.7, 10.0)
- moved U$4 5.38 mm to (34.8, 21.0), turned to 90 degrees
- moved IC5 4.32 mm to (73.5, 11.5)
- moved C5 3.53 mm to (65.8, 11.8)
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Connections:
- removed net ENCODER_1: U$5.1
- removed net ENCODER_2: U$5.2
- removed net HB_LEFT_1: U5.3, U5.7
- removed net HB_LEFT_2: U5.5, U5.9
- removed net HB_RIGHT_1: U2.3, U2.7
- removed net HB_RIGHT_2: U2.5, U2.9
- removed net PI_RX: U$6.31
- removed net PI_TX: U$6.33
- removed net RPI_ANALOG: R31.P$1, R6.P$1
- removed net V+: IC4.8, IC5.8
- removed net VOUT: IC4.7, IC5.7, R15.P$1, R28.P$1
- new net EDGE_LEFT: IC3.7, U$1.PC2
- new net EDGE_RIGHT: IC6.7, U$1.PC3
- new net ENCODER_LEFT_1: U$1.PB6, U$5.1
- new net ENCODER_LEFT_2: U$1.PB7, U$5.2
- new net ENCODER_RIGHT_1: U$1.PA0, U$7.1
- new net ENCODER_RIGHT_2: U$1.PA1, U$7.2
- new net IR_INT: IC2.7, U$1.PC1
- new net MOTOR_LEFT_1: U$1.PA8, U5.3, U5.7
- new net MOTOR_LEFT_2: U$1.PA9, U5.5, U5.9
- new net MOTOR_RIGHT_1: U$1.PA10, U2.3, U2.7
- new net MOTOR_RIGHT_2: U$1.PA11, U2.5, U2.9
- new net N$13: IC2.2, R35.2
- new net N$14: IC3.3, R15.P$1, U1.1
- new net N$15: IC3.2, R38.2
- new net N$17: R36.P$1, U6.3
- new net N$18: IC6.3, R34.P$1, U6.1
- new net N$19: IC6.2, R37.2
- new net N$3: R28.P$1, U1.3
- new net PI_ANALOG: R31.P$1, R6.P$1, U$1.PA2
- new net STM_RX: U$1.PC7, U$6.33
- new net STM_TX: U$1.PC6, U$6.31
- new net TAPE_LEFT: IC4.7, U$1.PB14
- new net TAPE_RIGHT: IC5.7, U$1.PB15
- net 5V_ANOLOG: now also C10.1, C11.1, C12.1, C28.1, C8.1, C9.1, IC2.8, IC3.8, IC4.8, IC5.8, IC6.8, R34.P$2, R35.3, R36.P$2, R37.3, R38.3; no longer IC4.5, IC5.5
- net GND: now also C10.2, C11.2, C12.2, C28.2, C8.2, C9.2, IC2.1, IC2.4, IC3.1, IC3.4, IC6.1, IC6.4, R35.1, R37.1, R38.1, U$7.3, U1.2, U1.4, U6.2, U6.4
- net IR_1: now also IC2.3, U$1.PA3
- net IR_2: now also U$1.PA4
- net PI_INT: now also U$1.PC0
- net SERVO_BASKET: now also U$1.PB0
- net SERVO_CLAW_1: now also U$1.PA6
- net SERVO_CLAW_2: now also U$1.PA7
Routing:
- net 6V_SERVO: track 40.3 -> 0.00 mm
- net MOTOR_RIGHT_1: track 0.00 -> 11.3 mm
- net HB_RIGHT_1: track 11.3 -> 0.00 mm
- net MOTOR_LEFT_1: track 0.00 -> 11.3 mm
- net HB_LEFT_1: track 11.3 -> 0.00 mm
- net MOTOR_RIGHT_2: track 0.00 -> 11.3 mm
- net HB_RIGHT_2: track 11.3 -> 0.00 mm
- net MOTOR_LEFT_2: track 0.00 -> 11.3 mm
- net HB_LEFT_2: track 11.3 -> 0.00 mm
