File: Electrical/modules/pcb/board.brd (EAGLE design)
At the start: 88.9 x 158.8 mm, 108 parts, among them IC1 OP-AMP, IC2 LM311N, IC3 LM311N, IC4 LM311N, IC5 LM311N, IC6 LM311N, M1 SERVO, M2 SERVO, M3 SERVO, U1 QRD1114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

Commit message: done
Parts:
- added FUSE: 2A, SparkFun-Resistors:AXIAL-0.3
- moved R9 21.9 mm to (73.7, 39.8), turned to 180 degrees
- moved R12 18.0 mm to (73.6, 35.2), turned to 0 degrees
- moved IC3 13.5 mm to (33.8, 32.9), turned to 0 degrees
- moved R11 12.1 mm to (74.2, 31.8)
- moved C9 11.5 mm to (6.70, 26.9)
- moved C8 10.9 mm to (14.8, 28.0)
- moved C10 10.3 mm to (46.2, 32.9), turned to 270 degrees
- moved R35 9.93 mm to (14.1, 35.9), turned to 180 degrees
- moved U4 7.56 mm to (83.6, 19.1)
- moved IC2 7.30 mm to (6.60, 34.0), turned to 90 degrees
- moved C11 4.39 mm to (41.4, 32.9), turned to 270 degrees
- moved C5 4.37 mm to (64.7, 16.0)
- moved IC5 4.34 mm to (72.4, 15.7)
- moved C1 4.33 mm to (64.0, 8.30)
- moved M1 4.32 mm to (62.7, 25.6), turned to 0 degrees
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Connections:
- new net FUSE: C20.1, C3.1, C4.1, C7.1, FUSE.P$2, U$3.OUT+
- net 5V_DIGITAL: now also FUSE.P$1; no longer C20.1, C3.1, C4.1, C7.1, U$3.OUT+
Routing:
- net 5V_ANOLOG: track 0.00 -> 239.5 mm
- net MOTOR_LEFT_1: track 11.3 -> 173.1 mm, vias 0 -> 2
- net PI_ANALOG: track 0.00 -> 154.9 mm
- net MOTOR_LEFT_2: track 11.3 -> 155.5 mm, vias 0 -> 1
- net IR_1: track 0.00 -> 133.1 mm
- net STM_RX: track 0.00 -> 114.3 mm
- net STM_TX: track 0.00 -> 112.0 mm
- net MOTOR_RIGHT_1: track 11.3 -> 109.5 mm, vias 0 -> 1
- net +5V: track 0.00 -> 81.9 mm
- net TAPE_LEFT: track 0.00 -> 77.2 mm
- net ENCODER_LEFT_1: track 0.00 -> 72.2 mm
- net MOTOR_RIGHT_2: track 11.3 -> 83.3 mm
- net N$18: track 0.00 -> 71.2 mm
- net SERVO_BASKET: track 0.00 -> 66.9 mm
- net SERVO_CLAW_2: track 0.00 -> 64.1 mm
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
Commit message: finalized circuit
Connections:
- new net N$32: U$1.1, U$1.2
- new net N$37: U$1.3, U$1.4
- net 5V_DIGITAL: now also U$6.2, U$6.4; no longer U$6.37, U$6.39
- net GND: now also U$6.14, U$6.20, U$6.25, U$6.30, U$6.34, U$6.39, U$6.6, U$6.9; no longer U$6.11, U$6.16, U$6.2, U$6.21, U$6.27, U$6.32, U$6.35, U$6.7
- net PI_INT: now also U$6.7; no longer U$6.4
- net R1: now also U$6.29; no longer U$6.19
- net R2: now also U$6.31; no longer U$6.23
- net R3: now also U$6.33; no longer U$6.25
- net R4: now also U$6.36; no longer U$6.26
- net R5: now also U$6.35; no longer U$6.28
- net R6: now also U$6.38; no longer U$6.30
- net R7: now also U$6.37; no longer U$6.29
- net R8: now also U$6.40; no longer U$6.34
- net STM_RX: now also U$6.8; no longer U$6.33
- net STM_TX: now also U$6.10; no longer U$6.31
Routing:
- net 5V_DIGITAL: track 70.3 -> 124.4 mm
- net STM_TX: track 112.0 -> 89.4 mm
- net STM_RX: track 114.3 -> 92.2 mm
- net R7: track 11.9 -> 4.44 mm
- net R5: track 13.0 -> 5.87 mm
- net PI_INT: track 43.2 -> 49.0 mm
- net IR_1: track 133.1 -> 127.4 mm, vias 0 -> 1
- net R6: track 13.4 -> 8.29 mm
- net R2: track 5.52 -> 9.42 mm
- net R4: track 9.52 -> 13.1 mm
- net R8: track 11.4 -> 7.97 mm
- net R1: track 6.58 -> 9.89 mm
- net 5V_ANOLOG: track 239.5 -> 242.7 mm
- net N$37: track 0.00 -> 2.54 mm
- net N$32: track 0.00 -> 2.54 mm
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
Commit message: updated cube, pcb
Parts:
- removed C20, C7: 1U, capacitor-wima:C5B5
- removed FUSE: 2A, SparkFun-Resistors:AXIAL-0.3
- removed LIPO_B: (no value), SparkFun-Connectors:DEANS
- added LIPO_BIG: (no value), SparkFun-Connectors:1X02
- added PI_FUSE: 2A, SparkFun-Resistors:AXIAL-0.3
- added STM_FUSE: 300mA, SparkFun-Resistors:AXIAL-0.3
- moved C4 17.1 mm to (61.8, 115.3), turned to 0 degrees
- moved C3 14.4 mm to (61.8, 121.5), turned to 0 degrees
- moved R16 13.9 mm to (83.1, 16.9)
- moved LIPO_SMALL_2 10.6 mm to (81.5, 105.5)
- moved U4 9.22 mm to (85.6, 10.1)
- moved R9 8.06 mm to (74.7, 31.8), flipped to the bottom, turned to 0 degrees
- moved R27 8.00 mm to (79.4, 9.70)
- moved C26 7.17 mm to (24.0, 130.1)
- moved U$11 6.77 mm to (58.2, 129.4)
- moved R12 6.32 mm to (75.6, 29.2), flipped to the bottom, turned to 180 degrees
- moved U$17 6.03 mm to (36.4, 128.7)
- moved C25 5.71 mm to (18.1, 127.6), turned to 0 degrees
- moved C15 5.10 mm to (77.0, 154.5)
- moved R11 5.10 mm to (75.2, 26.8), flipped to the bottom, turned to 0 degrees
- moved U$18 5.09 mm to (33.9, 137.0)
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Connections:
- removed net FUSE: C20.1, C3.1, C4.1, C7.1, FUSE.P$2, U$3.OUT+
- removed net N$14: IC3.3, R15.P$1, U1.1
- removed net N$18: IC6.3, R34.P$1, U6.1
- removed net N$28: IC4.3, R13.P$1, U3.1
- removed net N$31: IC5.3, R16.P$1, U4.1
- new net +3V3: QSD1.+, QSD2.+, U$1.+3V3
- new net ELA: IC3.3, R15.P$1, U$1.PC5, U1.1
- new net ERA: IC6.3, R34.P$1, U$1.PB1, U6.1
- new net PI_SUPPLY: PI_FUSE.P$1, U$6.2, U$6.4
- new net STM_SUPPLY: STM_FUSE.P$1, U$1.E5V
- new net TLA: IC4.3, R13.P$1, U$1.PC2, U3.1
- new net TRA: IC5.3, R16.P$1, U$1.PC4, U4.1
- net 5V_ANOLOG: no longer QSD1.+, QSD2.+
- net 5V_DIGITAL: now also C3.1, C4.1, PI_FUSE.P$2, STM_FUSE.P$2, U$3.OUT+; no longer FUSE.P$1, U$1.E5V, U$6.2, U$6.4
- net EDGE_LEFT: now also U$1.PD2; no longer U$1.PC2
- net GND: now also LIPO_BIG.1; no longer C20.2, C7.2, LIPO_B.-
- net IR_1: now also U$1.PA5; no longer U$1.PA3
- net LIPO_B_SUPPLY: now also LIPO_BIG.2; no longer LIPO_B.+
Routing:
- net PI_SUPPLY: track 0.00 -> 103.6 mm, vias 0 -> 3
- net ELA: track 0.00 -> 101.4 mm, vias 0 -> 2
- net 5V_DIGITAL: track 124.4 -> 23.3 mm
- net IR_1: track 127.4 -> 199.8 mm, vias 1 -> 2
- net N$18: track 71.2 -> 0.00 mm
- net STM_SUPPLY: track 0.00 -> 65.4 mm, vias 0 -> 1
- net ERA: track 0.00 -> 60.8 mm, vias 0 -> 1
- net +3V3: track 0.00 -> 57.4 mm
- net TLA: track 0.00 -> 56.9 mm, vias 0 -> 1
- net PI_ANALOG: track 154.9 -> 108.0 mm
- net TRA: track 0.00 -> 45.0 mm
- net SERVO_BASKET: track 66.9 -> 104.3 mm, vias 0 -> 2
- net LIPO_B_SUPPLY: track 31.4 -> 0.29 mm
- net GND: track 30.6 -> 0.00 mm
- net FUSE: track 29.2 -> 0.00 mm
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- added copper zone on layer 1, net 5V_ANALOG
Other:
- outline, holes or cut-outs redrawn
