File: Electrical/modules/pcb/board.brd (EAGLE design)
At the start: 88.9 x 158.8 mm, 108 parts, among them IC1 OP-AMP, IC2 LM311N, IC3 LM311N, IC4 LM311N, IC5 LM311N, IC6 LM311N, M1 SERVO, M2 SERVO, M3 SERVO, U1 QRD1114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

Commit message: fix
Routing:
- net N$37: track 5.08 -> 2.54 mm
- net N$32: track 5.08 -> 2.54 mm
Changed lines of the file:
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@@
 <wire x1="29.5" y1="23" x2="29.5698" y2="23" width="0.1524" layer="1"/>
-</signal>
-<signal name="N$32">
-<contactref element="U$1" pad="2"/>
-<contactref element="U$1" pad="1"/>
-<wire x1="22" y1="102.12" x2="22" y2="104.66" width="0.1524" layer="1"/>
-</signal>
-<signal name="N$37">
-<contactref element="U$1" pad="4"/>
-<contactref element="U$1" pad="3"/>
-<wire x1="85.5" y1="102.12" x2="85.5" y2="104.66" width="0.1524" layer="1"/>
 </signal>
 </signals>
