File: Electrical/modules/pcb/board.sch (EAGLE design)
At the start: 21 parts, among them IC1 OP-AMP, IC2 LM311N, U1 UA7805CKCS, U2 UA7805CKCS

Commit message: pcb
Parts:
- removed C3: 0.1uF, SparkFun-Capacitors:0.1UF-KIT-EZ-50V-20%
- removed C4: 0.33uF, SparkFun-Capacitors:0.1UF-KIT-EZ-50V-20%
- removed J1: (no value), SparkFun-Connectors:CONN_02
- removed U2: UA7805CKCS, regulator:UA7805CKCS
- added C10, C13, C14, C15, C16, C17, C18, C8: 0.1uF, SparkFun-Capacitors:0.1UF-KIT-EZ-50V-20%
- added C11, C9: 100nf, Seeed-Capacitor:DIP-CERAMIC-DISC-100NF-50V-Y5V(D5.0MM)
- added C12, C19: 1uF, SparkFun-Capacitors:0.1UF-KIT-EZ-50V-20%
- added J4, J6: (no value), SparkFun-Connectors:CONN_02
- added Q1, Q2, Q5, Q6: IRF3505, IRF3505:IRF3205PBF
- added R17, R18, R22, R24, R37, R38, R42, R44: 10k, SparkFun-Resistors:10KOHM-HORIZ-1/4W-1%
- added R19, R21, R23, R26, R39, R41, R43, R46: 100, SparkFun-Resistors:10KOHM-HORIZ-1/4W-1%
- added R20, R25, R40, R45: 33k, SparkFun-Resistors:10KOHM-HORIZ-1/4W-1%
- added T13, T14, T5, T6: 2N3904, transistor:2N3904
- added T15, T16, T7, T8: 2N3906BU, 2N3906:2N3906BU
- added U10, U5, U6, U9: HUF75321, HUF75321:STP45N65M5
Connections:
- removed net 5V_IC: C1.1, C5.1, C6.1, C7.1, IC1G3.P$V+, IC2.V+, QSD1.+, R1.A, R4.2, R6.2, U1.OUT
- removed net 5V_STM: C3.1, U$1.P$35, U2.OUT
- removed net V_IN: C4.1, J1.2, U2.IN
- new net 5V_SUPPLY: C1.1, C5.1, C6.1, C7.1, IC1G3.P$V+, IC2.V+, QSD1.+, R1.A, R4.2, R6.2, U$1.P$35, U1.OUT
- new net LEFT_1: T13.B
- new net LEFT_2: T14.B
- new net N$17: Q1.G, R18.1, R19.2, R25.2
- new net N$18: R19.1, T5.C
- new net N$19: R23.1, T6.C
- new net N$20: R17.2, R21.1, U6.1
- new net N$21: R21.2, T7.C
- new net N$22: R20.2, T7.B
- new net N$23: R24.2, R26.1, U5.1
- new net N$24: R26.2, T8.C
- new net N$25: R25.1, T8.B
- new net N$26: Q2.G, R20.1, R22.1, R23.2
- new net N$27: C9.2, J4.1, Q2.D, U5.2
- new net N$41: Q5.G, R38.1, R39.2, R45.2
- new net N$42: R39.1, T13.C
- new net N$43: R43.1, T14.C
- new net N$44: R37.2, R41.1, U10.1
- new net N$45: R41.2, T15.C
- new net N$46: R40.2, T15.B
- new net N$47: R44.2, R46.1, U9.1
- new net N$48: R46.2, T16.C
- new net N$49: R45.1, T16.B
- new net N$50: Q6.G, R40.1, R42.1, R43.2
- new net N$51: C11.2, J6.1, Q6.D, U9.2
- new net N$8: C9.1, J4.2, Q1.D, U6.2
- new net N$9: C11.1, J6.2, Q5.D, U10.2
- new net RIGHT_1: T5.B
- new net RIGHT_2: T6.B
- new net VCC: C10.1, C12.1, C13.1, C14.1, C15.1, C16.1, C17.1, C18.1, C19.1, C8.1, Q1.S, Q2.S, Q5.S, Q6.S, R18.2, R22.2, R38.2, R42.2, T15.E, T16.E, T7.E, T8.E
- net GND: now also C10.2, C12.2, C13.2, C14.2, C15.2, C16.2, C17.2, C18.2, C19.2, C8.2, R17.1, R24.1, R37.1, R44.1, T13.E, T14.E, T5.E, T6.E, U10.3, U5.3, U6.3, U9.3; no longer C3.2, C4.2, J1.1, U2.COM
Other:
- note added: "TODO: Confirm cricuit"
- note added: "TODO: Test hbridges with stm Assign STM pints (pull ups?)"

Commit message: circuit updates
Parts:
- removed R2: 20k, SparkFun-Resistors:10KOHM-HORIZ-1/4W-1%
- added C20: 0.33uF, SparkFun-Capacitors:0.1UF-KIT-EZ-50V-20%
- added C21, C23, C4: 0.1uF, SparkFun-Capacitors:0.1UF-KIT-EZ-50V-20%
- added C22, C24: 1uF, SparkFun-Capacitors:0.1UF-KIT-EZ-50V-20%
- added C3: 470pF, SparkFun-Capacitors:0.1UF-KIT-EZ-50V-20%
- added D1, D2: 1N4004, adafruit:1N4004
- added IC4, IC5: LM311N, linear:LM311N
- added J1: (no value), SparkFun-Connectors:BATTERY_CONN_DEANS
- added R10: (no value), resistor:R-TRIMMT93YA
- added R13, R15, R16, R28: 47k, rcl:R-US_0204/5
- added R14, R27: 300, rcl:R-US_0204/5
- added R7, R8, R9: 10k, SparkFun-Resistors:10KOHM-HORIZ-1/4W-1%
- added U2: UA7805CKCS, regulator:UA7805CKCS
- added U3, U4: QRD1114, SparkFun-Sensors:QRD1114
- added VR2, VR3: 5k, SparkFun-Resistors:TRIMPOT-SMD-5MM-CLOSED-1/4W-20%
- R3: value 20k -> 33k
Connections:
- net VCC renamed LIPO_SUPPLY
- removed net 5V_SUPPLY: C1.1, C5.1, C6.1, C7.1, IC1G3.P$V+, IC2.V+, QSD1.+, R1.A, R4.2, R6.2, U$1.P$35, U1.OUT
- removed net N$5: IC1G2.-IN, R2.1, R4.1
- new net 5V_AC: C1.1, C21.1, C22.1, C23.1, C24.1, C5.1, C6.1, C7.1, D1.A, IC1G3.P$V+, IC2.V+, IC4.ON, IC5.ON, QSD1.+, R1.A, R13.2, R14.2, R15.2, R16.2, R27.2, R28.2, U1.OUT, VR2.CCW, VR3.CCW
- new net 5V_DC: C4.1, D2.A, U$1.P$35, U2.OUT
- new net N$10: R9.2, T14.B
- new net N$11: R8.1, T13.B
- new net N$14: R7.2, T6.B
- new net N$15: R6.1, T5.B
- new net N$16: R14.1, U3.A
- new net N$28: IC4.-IN, R13.1, U3.C
- new net N$29: IC4.+IN, VR2.WIPER
- new net N$30: R27.1, U4.A
- new net N$31: IC5.-IN, R16.1, U4.C
- new net N$32: IC5.+IN, VR3.WIPER
- new net N$7: IC1G1.-IN, IC1G1.OUT, R3.1
- new net VOUT: IC4.OUT, IC5.OUT, R15.1, R28.1
- new net V_IN2: C20.1, D2.C, J1.+, U2.IN
- net GND: now also C20.2, C21.2, C22.2, C23.2, C24.2, C3.2, C4.2, IC4.GND, IC4.V-, IC5.GND, IC5.V-, J1.-, R4.2, U2.COM, U3.E, U3.K, U4.E, U4.K, VR2.CW, VR3.CW
- net LEFT_1: now also R8.2; no longer T13.B
- net LEFT_2: now also R9.1; no longer T14.B
- net N$2: now also C3.1; no longer IC1G1.OUT
- net N$3: now also R10.S; no longer R2.2
- net N$4: now also IC1G2.-IN, R10.A, R4.1; no longer IC1G1.-IN, R3.1, R6.1
- net RIGHT_1: now also R6.2; no longer T5.B
- net RIGHT_2: now also R7.1; no longer T6.B
- net V_IN1: now also D1.C
Other:
- note added: "TODO: Assign STM pints with pull ups"
- note removed: "TODO: Confirm cricuit"
- note removed: "TODO: Test OpAmp configuration works. Assign pin on stm"
- note removed: "TODO: Test hbridges with stm Assign STM pints (pull ups?)"
- moved on the sheet: IC1G1, IC1G2, R3, R4, R6

Commit message: updates
Parts:
- removed C10, C13, C14, C15, C16, C17, C18, C8: 0.1uF, SparkFun-Capacitors:0.1UF-KIT-EZ-50V-20%
- removed C11, C9: 100nf, Seeed-Capacitor:DIP-CERAMIC-DISC-100NF-50V-Y5V(D5.0MM)
- removed C12, C19: 1uF, SparkFun-Capacitors:0.1UF-KIT-EZ-50V-20%
- removed D2: 1N4004, adafruit:1N4004
- removed IC2: LM311N, linear:LM311N
- removed J1: (no value), SparkFun-Connectors:BATTERY_CONN_DEANS
- removed J2, J4, J6: (no value), SparkFun-Connectors:CONN_02
- removed Q1, Q2, Q5, Q6: IRF3505, IRF3505:IRF3205PBF
- removed R17, R18, R22, R24, R37, R38, R42, R44, R6, R7, R8, R9: 10k, SparkFun-Resistors:10KOHM-HORIZ-1/4W-1%
- removed R19, R21, R23, R26, R39, R41, R43, R46: 100, SparkFun-Resistors:10KOHM-HORIZ-1/4W-1%
- removed R20, R25, R40, R45: 33k, SparkFun-Resistors:10KOHM-HORIZ-1/4W-1%
- removed T13, T14, T5, T6: 2N3904, transistor:2N3904
- removed T15, T16, T7, T8: 2N3906BU, 2N3906:2N3906BU
- removed U1, U2: UA7805CKCS, regulator:UA7805CKCS
- removed U10, U5, U6, U9: HUF75321, HUF75321:STP45N65M5
- added LIPO_B: (no value), SparkFun-Connectors:BATTERY_CONN_DEANS
- added LIPO_SMALL_1, LIPO_SMALL_2: (no value), SparkFun-Connectors:CONN_02
- added QSD2: (no value), Seeed-LED:DIP-LED-GREEN-GREEN(2P-D5MM)
- added R2: 10k, SparkFun-Resistors:10KOHM-HORIZ-1/4W-1%
- added U$2, U$3: DC-DC-STEP-DOWN-LM2596, diy-modules:DC-DC-STEP-DOWN-LM2596
- added U$4: UA7805, TO220:UA7805
- C20: value 0.33uF -> 1U; device SparkFun-Capacitors:0.1UF-KIT-EZ-50V-20% -> capacitor-wima:C5/5
- C3: value 470pF -> 1U; device SparkFun-Capacitors:0.1UF-KIT-EZ-50V-20% -> capacitor-wima:C5/5
- C4, C7: value 0.1uF -> 1U; device SparkFun-Capacitors:0.1UF-KIT-EZ-50V-20% -> capacitor-wima:C5/5
- R1: value (none) -> 1k; device resistor:R-TRIMMT93YA -> SparkFun-Resistors:1KOHM-HORIZ-1/4W-5%
- R10: value (none) -> 100k
- R3: value 33k -> 100k; device SparkFun-Resistors:10KOHM-HORIZ-1/4W-1% -> resistor:R-TRIMMT93YA
Connections:
- removed net 5V_AC: C1.1, C21.1, C22.1, C23.1, C24.1, C5.1, C6.1, C7.1, D1.A, IC1G3.P$V+, IC2.V+, IC4.ON, IC5.ON, QSD1.+, R1.A, R13.2, R14.2, R15.2, R16.2, R27.2, R28.2, U1.OUT, VR2.CCW, VR3.CCW
- removed net GPIO_IR: IC2.OUT
- removed net LEFT_1: R8.2
- removed net LEFT_2: R9.1
- removed net LIPO_SUPPLY: C10.1, C12.1, C13.1, C14.1, C15.1, C16.1, C17.1, C18.1, C19.1, C8.1, Q1.S, Q2.S, Q5.S, Q6.S, R18.2, R22.2, R38.2, R42.2, T15.E, T16.E, T7.E, T8.E
- removed net N$10: R9.2, T14.B
- removed net N$11: R8.1, T13.B
- removed net N$14: R7.2, T6.B
- removed net N$15: R6.1, T5.B
- removed net N$17: Q1.G, R18.1, R19.2, R25.2
- removed net N$18: R19.1, T5.C
- removed net N$19: R23.1, T6.C
- removed net N$20: R17.2, R21.1, U6.1
- removed net N$21: R21.2, T7.C
- removed net N$22: R20.2, T7.B
- removed net N$23: R24.2, R26.1, U5.1
- removed net N$24: R26.2, T8.C
- removed net N$25: R25.1, T8.B
- removed net N$26: Q2.G, R20.1, R22.1, R23.2
- removed net N$27: C9.2, J4.1, Q2.D, U5.2
- removed net N$41: Q5.G, R38.1, R39.2, R45.2
- removed net N$42: R39.1, T13.C
- removed net N$43: R43.1, T14.C
- removed net N$44: R37.2, R41.1, U10.1
- removed net N$45: R41.2, T15.C
- removed net N$46: R40.2, T15.B
- removed net N$47: R44.2, R46.1, U9.1
- removed net N$48: R46.2, T16.C
- removed net N$49: R45.1, T16.B
- removed net N$50: Q6.G, R40.1, R42.1, R43.2
- removed net N$51: C11.2, J6.1, Q6.D, U9.2
- removed net N$7: IC1G1.-IN, IC1G1.OUT, R3.1
- removed net N$8: C9.1, J4.2, Q1.D, U6.2
- removed net N$9: C11.1, J6.2, Q5.D, U10.2
- removed net RIGHT_1: R6.2
- removed net RIGHT_2: R7.1
- removed net V_IN2: C20.1, D2.C, J1.+, U2.IN
- new net 5V_ANOLOG: C1.1, C21.1, C22.1, C23.1, C24.1, C5.1, C6.1, D1.A, IC1G3.P$V+, IC4.ON, IC5.ON, QSD1.+, QSD2.+, R13.2, R14.2, R15.2, R16.2, R27.2, R28.2, U$4.OUT, VR2.CCW, VR3.CCW
- new net 5V_DIGITAL: C20.1, C3.1, C4.1, C7.1, U$3.OUT+
- new net 6V_SERVO: U$2.OUT+
- new net IR_1: IC1G2.OUT, R10.S
- new net IR_3: IC1G1.OUT, R3.S
- new net LIPO_B_GND: LIPO_B.-, U$3.IN-
- new net LIPO_B_SUPPLY: LIPO_B.+, U$3.IN+
- new net OUTPUT2: IC1G1.+IN, QSD2.-, R1.2
- net 5V_DC: no longer C4.1, D2.A, U2.OUT
- net GND: now also LIPO_SMALL_1.1, R1.1, R2.2, U$2.OUT-, U$3.OUT-, U$4.COM; no longer C10.2, C12.2, C13.2, C14.2, C15.2, C16.2, C17.2, C18.2, C19.2, C8.2, IC2.GND, IC2.V-, J1.-, J2.1, R1.E, R17.1, R24.1, R37.1, R44.1, T13.E, T14.E, T5.E, T6.E, U1.COM, U10.3, U2.COM, U5.3, U6.3, U9.3
- net N$1: now also LIPO_SMALL_2.2, U$2.IN+; no longer IC2.+IN, R1.S
- net N$2: now also IC1G1.-IN, R2.1, R3.A; no longer C3.1, IC1G2.+IN, R3.2
- net N$3: now also LIPO_SMALL_2.1, U$2.IN-; no longer IC1G2.OUT, IC2.-IN, R10.S
- net OUTPUT1: now also IC1G2.+IN; no longer IC1G1.+IN
- net V_IN1: now also LIPO_SMALL_1.2, U$4.IN; no longer J2.2, U1.IN
Other:
- note added: "2x(85 + 250)/5 = 130 mA"
- note added: "431/5 = 107 mA"
- note added: "Big Lipo: Motors, STM and Pi via Switching regulator Small Lipo: Servos via switching regulator Small Lipo: ICs via linear regulator"
- note added: "IR Sensor"
- note added: "Power"
- note added: "STM"
- note added: "TODO: Assign STM pints (no pull up needed)"
- note added: "Tape Followers"
- moved on the sheet: C1, C2, C20, C3, C4, C5, C6, C7, D1, IC1G1, IC1G2, IC1G3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

Commit message: updates
Parts:
- added M1, M2, M3: SERVO, SparkFun-Electromechanical:SERVO
- added R11, R12, R9: 1k, SparkFun-Resistors:1KOHM-HORIZ-1/4W-5%
- added U$5: ENCODER, TO220:ENCODER
- added U$6: RPI3, Raspberry_Pi_3:RPI3
Connections:
- net IR_3 renamed IR_2
- removed net 5V_DC: U$1.P$35
- new net +5V: R11.2, R12.2, R9.2, U$1.P$29
- new net ENCODER_1: U$5.1
- new net ENCODER_2: U$5.2
- new net SERVO_BASKET: M3.SIG
- new net SERVO_CLAW_1: M2.SIG
- new net SERVO_CLAW_2: M1.SIG
- net 5V_DIGITAL: now also U$1.P$35
- net 6V_SERVO: now also M1.V+, M2.V+, M3.V+, R11.1, R12.1, R9.1
- net GND: now also M1.GND, M2.GND, M3.GND, U$5.GND
Other:
- note added: "Servos"
- note added: "TODO: Assign pins"
- note added: "TODO: Assign pins, with open drain"
- moved on the sheet: C1, C2, C20, C21, C22, C23, C24, C3, C4, C5, C6, C7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

Commit message: updates
Parts:
- removed VR2, VR3: 5k, SparkFun-Resistors:TRIMPOT-SMD-5MM-CLOSED-1/4W-20%
- added C13, C15, C18, C25: 1uF, SparkFun-Capacitors:0.1UF-KIT-EZ-50V-20%
- added C14, C16, C17, C19, C26, C27: 0.1uF, SparkFun-Capacitors:0.1UF-KIT-EZ-50V-20%
- added D4, D5, D6, D7: 15V, diode:ZENER-DIODEDO41Z10
- added J2, J3: (no value), SparkFun-Connectors:CONN_02
- added R17, R18, R19, R20, R21, R22, R23, R24, R25, R26, R29, R30, R31, R6, R7, R8: 1k, SparkFun-Resistors:1KOHM-HORIZ-1/4W-1%
- added R32, R33: 10k, resistor:R-TRIMMT93YA
- added U$11, U$12, U$13, U$14, U$15, U$16, U$17, U$18: HUF75321, TO220:HUF75321
- added U2, U5: LT1161CNPBF, LT1161NC:LT1161CNPBF
- R13, R15, R16, R28: value 47k -> 1k; device rcl:R-US_0204/5 -> SparkFun-Resistors:1KOHM-HORIZ-1/4W-1%
- R14, R27: value 300 -> 1k; device rcl:R-US_0204/5 -> SparkFun-Resistors:1KOHM-HORIZ-1/4W-1%
Connections:
- removed net N$32: IC5.+IN, VR3.WIPER
- new net HB_LEFT_1: U5.INPUT1, U5.INPUT3
- new net HB_LEFT_2: U5.INPUT2, U5.INPUT4
- new net HB_RIGHT_1: U2.INPUT1, U2.INPUT3
- new net HB_RIGHT_2: U2.INPUT2, U2.INPUT4
- new net N$10: R17.1, R26.1, R29.2
- new net N$11: R29.1, R30.2, R8.1
- new net N$12: R30.1, R31.2, R7.1
- new net N$20: U$11.G, U2.GATE1
- new net N$21: U$12.G, U2.GATE2
- new net N$22: D5.C, U$14.G, U2.GATE3
- new net N$23: D4.C, U$13.G, U2.GATE4
- new net N$24: C17.2, J2.1, U$12.S, U$14.D
- new net N$25: C17.1, J2.2, U$11.S, U$13.D
- new net N$26: U$15.G, U5.GATE1
- new net N$27: U$16.G, U5.GATE2
- new net N$33: D7.C, U$18.G, U5.GATE3
- new net N$34: D6.C, U$17.G, U5.GATE4
- new net N$35: C27.2, J3.1, U$16.S, U$18.D
- new net N$36: C27.1, J3.2, U$15.S, U$17.D
- new net N$5: R21.1, R22.1, R23.2
- new net N$6: IC5.+IN, R32.S
- new net N$7: R20.1, R23.1, R24.2
- new net N$8: R19.1, R24.1, R25.2
- new net N$9: R18.1, R25.1, R26.2
- new net PI_INT: U$6.P$4
- new net PI_RX: U$6.P$31
- new net PI_TX: U$6.P$33
- new net R1: R21.2, U$6.P$19
- new net R2: R20.2, U$6.P$23
- new net R3: R19.2, U$6.P$25
- new net R4: R18.2, U$6.P$26
- new net R5: R17.2, U$6.P$28
- new net R6: R8.2, U$6.P$30
- new net R7: R7.2, U$6.P$29
- new net R8: R6.2, U$6.P$34
- new net RPI_ANALOG: R31.1, R6.1
- new net VCC: C18.1, C19.1, C25.1, C26.1, U$15.D, U$16.D, U5.SENSE1, U5.SENSE2, U5.SENSE3, U5.SENSE4, U5.V+, U5.V+_2
- net 5V_ANOLOG: now also R32.A, R33.A; no longer VR2.CCW, VR3.CCW
- net 5V_DIGITAL: now also U$6.P$37, U$6.P$39
- net GND: now also C15.2, C16.2, C18.2, C19.2, C25.2, C26.2, D6.A, D7.A, R22.2, R32.E, R33.E, U$17.S, U$18.S, U$6.P$11, U$6.P$16, U$6.P$2, U$6.P$21, U$6.P$27, U$6.P$32, U$6.P$35, U$6.P$7, U5.GND, U5.GND_2; no longer VR2.CW, VR3.CW
- net LIPO_B_GND: now also C13.2, C14.2, D4.A, D5.A, U$13.S, U$14.S, U2.GND, U2.GND_2
- net LIPO_B_SUPPLY: now also C13.1, C14.1, C15.1, C16.1, U$11.D, U$12.D, U2.SENSE1, U2.SENSE2, U2.SENSE3, U2.SENSE4, U2.V+, U2.V+_2
- net N$29: now also R33.S; no longer VR2.WIPER
Other:
- note added: "Left H-Bridge"
- note added: "Right H-Bridge"
- note added: "TODO: Assign pins on stm. Rx and tx switch."

Commit message: updates
Connections:
- removed net LIPO_B_GND: C13.2, C14.2, D4.A, D5.A, LIPO_B.-, U$13.S, U$14.S, U$3.IN-, U2.GND, U2.GND_2
- removed net N$3: LIPO_SMALL_2.1, U$2.IN-
- removed net VCC: C18.1, C19.1, C25.1, C26.1, U$15.D, U$16.D, U5.SENSE1, U5.SENSE2, U5.SENSE3, U5.SENSE4, U5.V+, U5.V+_2
- net 6V_SERVO: no longer R11.1, R12.1, R9.1
- net GND: now also C13.2, C14.2, D4.A, D5.A, LIPO_B.-, LIPO_SMALL_2.1, U$13.S, U$14.S, U$2.IN-, U$3.IN-, U2.GND, U2.GND_2
- net LIPO_B_SUPPLY: now also C18.1, C19.1, C25.1, C26.1, U$15.D, U$16.D, U5.SENSE1, U5.SENSE2, U5.SENSE3, U5.SENSE4, U5.V+, U5.V+_2
- net SERVO_BASKET: now also R12.1
- net SERVO_CLAW_1: now also R11.1
- net SERVO_CLAW_2: now also R9.1
Other:
- note added: "Encoder"
- note added: "Raspberry Pi"
- moved on the sheet: R11, R12, R9

Commit message: almost there
Parts:
- R17, R18, R19, R20, R21, R22, R6, R7, R8: value 1k -> 100k
- R23, R24, R25, R26, R29, R30, R31: value 1k -> 50k
Other:
- note added: "Complete: Intrrupts from GPIO and reading same singal? Comparators for ir sensors to trigger interrupts? Confirm STM pinout"
Changed lines of the file:
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@@
 <part name="U$6" library="Raspberry_Pi_3" deviceset="RPI3" device=""/>
 <part name="SUPPLY5" library="supply2" library_urn="urn:adsk.eagle:library:372" deviceset="GND" device=""/>
-<part name="R6" library="SparkFun-Resistors" library_urn="urn:adsk.eagle:library:532" deviceset="1KOHM" device="-HORIZ-1/4W-1%" package3d_urn="urn:adsk.eagle:package:39658/1" value="1k"/>
-<part name="R7" library="SparkFun-Resistors" library_urn="urn:adsk.eagle:library:532" deviceset="1KOHM" device="-HORIZ-1/4W-1%" package3d_urn="urn:adsk.eagle:package:39658/1" value="1k"/>
-<part name="R8" library="SparkFun-Resistors" library_urn="urn:adsk.eagle:library:532" deviceset="1KOHM" device="-HORIZ-1/4W-1%" package3d_urn="urn:adsk.eagle:package:39658/1" value="1k"/>
-<part name="R17" library="SparkFun-Resistors" library_urn="urn:adsk.eagle:library:532" deviceset="1KOHM" device="-HORIZ-1/4W-1%" package3d_urn="urn:adsk.eagle:package:39658/1" value="1k"/>
-<part name="R18" library="SparkFun-Resistors" library_urn="urn:adsk.eagle:library:532" deviceset="1KOHM" device="-HORIZ-1/4W-1%" package3d_urn="urn:adsk.eagle:package:39658/1" value="1k"/>
-<part name="R19" library="SparkFun-Resistors" library_urn="urn:adsk.eagle:library:532" deviceset="1KOHM" device="-HORIZ-1/4W-1%" package3d_urn="urn:adsk.eagle:package:39658/1" value="1k"/>
-<part name="R20" library="SparkFun-Resistors" library_urn="urn:adsk.eagle:library:532" deviceset="1KOHM" device="-HORIZ-1/4W-1%" package3d_urn="urn:adsk.eagle:package:39658/1" value="1k"/>
-<part name="R21" library="SparkFun-Resistors" library_urn="urn:adsk.eagle:library:532" deviceset="1KOHM" device="-HORIZ-1/4W-1%" package3d_urn="urn:adsk.eagle:package:39658/1" value="1k"/>
-<part name="R22" library="SparkFun-Resistors" library_urn="urn:adsk.eagle:library:532" deviceset="1KOHM" device="-HORIZ-1/4W-1%" package3d_urn="urn:adsk.eagle:package:39658/1" value="1k"/>
-<part name="R23" library="SparkFun-Resistors" library_urn="urn:adsk.eagle:library:532" deviceset="1KOHM" device="-HORIZ-1/4W-1%" package3d_urn="urn:adsk.eagle:package:39658/1" value="1k"/>
-<part name="R24" library="SparkFun-Resistors" library_urn="urn:adsk.eagle:library:532" deviceset="1KOHM" device="-HORIZ-1/4W-1%" package3d_urn="urn:adsk.eagle:package:39658/1" value="1k"/>
-<part name="R25" library="SparkFun-Resistors" library_urn="urn:adsk.eagle:library:532" deviceset="1KOHM" device="-HORIZ-1/4W-1%" package3d_urn="urn:adsk.eagle:package:39658/1" value="1k"/>
-<part name="R26" library="SparkFun-Resistors" library_urn="urn:adsk.eagle:library:532" deviceset="1KOHM" device="-HORIZ-1/4W-1%" package3d_urn="urn:adsk.eagle:package:39658/1" value="1k"/>
-<part name="R29" library="SparkFun-Resistors" library_urn="urn:adsk.eagle:library:532" deviceset="1KOHM" device="-HORIZ-1/4W-1%" package3d_urn="urn:adsk.eagle:package:39658/1" value="1k"/>
-<part name="R30" library="SparkFun-Resistors" library_urn="urn:adsk.eagle:library:532" deviceset="1KOHM" device="-HORIZ-1/4W-1%" package3d_urn="urn:adsk.eagle:package:39658/1" value="1k"/>
-<part name="R31" library="SparkFun-Resistors" library_urn="urn:adsk.eagle:library:532" deviceset="1KOHM" device="-HORIZ-1/4W-1%" package3d_urn="urn:adsk.eagle:package:39658/1" value="1k"/>
+<part name="R6" library="SparkFun-Resistors" library_urn="urn:adsk.eagle:library:532" deviceset="1KOHM" device="-HORIZ-1/4W-1%" package3d_urn="urn:adsk.eagle:package:39658/1" value="100k"/>
+<part name="R7" library="SparkFun-Resistors" library_urn="urn:adsk.eagle:library:532" deviceset="1KOHM" device="-HORIZ-1/4W-1%" package3d_urn="urn:adsk.eagle:package:39658/1" value="100k"/>
+<part name="R8" library="SparkFun-Resistors" library_urn="urn:adsk.eagle:library:532" deviceset="1KOHM" device="-HORIZ-1/4W-1%" package3d_urn="urn:adsk.eagle:package:39658/1" value="100k"/>
+<part name="R17" library="SparkFun-Resistors" library_urn="urn:adsk.eagle:library:532" deviceset="1KOHM" device="-HORIZ-1/4W-1%" package3d_urn="urn:adsk.eagle:package:39658/1" value="100k"/>
+<part name="R18" library="SparkFun-Resistors" library_urn="urn:adsk.eagle:library:532" deviceset="1KOHM" device="-HORIZ-1/4W-1%" package3d_urn="urn:adsk.eagle:package:39658/1" value="100k"/>
+<part name="R19" library="SparkFun-Resistors" library_urn="urn:adsk.eagle:library:532" deviceset="1KOHM" device="-HORIZ-1/4W-1%" package3d_urn="urn:adsk.eagle:package:39658/1" value="100k"/>
+<part name="R20" library="SparkFun-Resistors" library_urn="urn:adsk.eagle:library:532" deviceset="1KOHM" device="-HORIZ-1/4W-1%" package3d_urn="urn:adsk.eagle:package:39658/1" value="100k"/>
+<part name="R21" library="SparkFun-Resistors" library_urn="urn:adsk.eagle:library:532" deviceset="1KOHM" device="-HORIZ-1/4W-1%" package3d_urn="urn:adsk.eagle:package:39658/1" value="100k"/>
+<part name="R22" library="SparkFun-Resistors" library_urn="urn:adsk.eagle:library:532" deviceset="1KOHM" device="-HORIZ-1/4W-1%" package3d_urn="urn:adsk.eagle:package:39658/1" value="100k"/>
+<part name="R23" library="SparkFun-Resistors" library_urn="urn:adsk.eagle:library:532" deviceset="1KOHM" device="-HORIZ-1/4W-1%" package3d_urn="urn:adsk.eagle:package:39658/1" value="50k"/>
+<part name="R24" library="SparkFun-Resistors" library_urn="urn:adsk.eagle:library:532" deviceset="1KOHM" device="-HORIZ-1/4W-1%" package3d_urn="urn:adsk.eagle:package:39658/1" value="50k"/>
+<part name="R25" library="SparkFun-Resistors" library_urn="urn:adsk.eagle:library:532" deviceset="1KOHM" device="-HORIZ-1/4W-1%" package3d_urn="urn:adsk.eagle:package:39658/1" value="50k"/>
+<part name="R26" library="SparkFun-Resistors" library_urn="urn:adsk.eagle:library:532" deviceset="1KOHM" device="-HORIZ-1/4W-1%" package3d_urn="urn:adsk.eagle:package:39658/1" value="50k"/>
+<part name="R29" library="SparkFun-Resistors" library_urn="urn:adsk.eagle:library:532" deviceset="1KOHM" device="-HORIZ-1/4W-1%" package3d_urn="urn:adsk.eagle:package:39658/1" value="50k"/>
+<part name="R30" library="SparkFun-Resistors" library_urn="urn:adsk.eagle:library:532" deviceset="1KOHM" device="-HORIZ-1/4W-1%" package3d_urn="urn:adsk.eagle:package:39658/1" value="50k"/>
+<part name="R31" library="SparkFun-Resistors" library_urn="urn:adsk.eagle:library:532" deviceset="1KOHM" device="-HORIZ-1/4W-1%" package3d_urn="urn:adsk.eagle:package:39658/1" value="50k"/>
 <part name="U2" library="LT1161NC" deviceset="LT1161CNPBF" device=""/>
 <part name="C13" library="SparkFun-Capacitors" library_urn="urn:adsk.eagle:library:510" deviceset="0.1UF" device="-KIT-EZ-50V-20%" package3d_urn="urn:adsk.eagle:package:37428/1" value="1uF"/>
@@
 <text x="160.02" y="149.86" size="1.778" layer="94">Encoder</text>
 <text x="210.82" y="309.88" size="1.778" layer="94">Raspberry Pi</text>
+<text x="579.12" y="231.14" size="1.778" layer="91">Complete:
+Intrrupts from GPIO and reading same singal?
+Comparators for ir sensors to trigger interrupts?
+Confirm STM pinout
+</text>
 </plain>
 <instances>
