File: Electrical/modules/pcb/board.sch (EAGLE design)
At the start: 91 parts, among them IC1 OP-AMP, IC4 LM311N, IC5 LM311N, M1 SERVO, M2 SERVO, M3 SERVO, U2 LT1161CNPBF, U3 QRD1114, U4 QRD1114, U5 LT1161CNPBF

Commit message: updates
Parts:
- added C10, C12, C8: 0.1uF, SparkFun-Capacitors:0.1UF-KIT-EZ-50V-20%
- added C11, C28, C9: 1uF, SparkFun-Capacitors:0.1UF-KIT-EZ-50V-20%
- added IC2, IC3, IC6: LM311N, linear:LM311N
- added R34: 47k, SparkFun-Resistors:1KOHM-HORIZ-1/4W-1%
- added R35, R37, R38: 10k, resistor:R-TRIMMT93YA
- added R36: 300, SparkFun-Resistors:1KOHM-HORIZ-1/4W-1%
- added U$7: ENCODER, TO220:ENCODER
- added U1, U6: QRD1114, SparkFun-Sensors:QRD1114
- R13, R15, R16: value 1k -> 47k
- R14, R27, R28: value 1k -> 300
Connections:
- removed net ENCODER_1: U$5.1
- removed net ENCODER_2: U$5.2
- removed net HB_LEFT_1: U5.INPUT1, U5.INPUT3
- removed net HB_LEFT_2: U5.INPUT2, U5.INPUT4
- removed net HB_RIGHT_1: U2.INPUT1, U2.INPUT3
- removed net HB_RIGHT_2: U2.INPUT2, U2.INPUT4
- removed net PI_RX: U$6.P$31
- removed net PI_TX: U$6.P$33
- removed net RPI_ANALOG: R31.1, R6.1
- removed net VOUT: IC4.OUT, IC5.OUT, R15.1, R28.1
- new net EDGE_LEFT: IC3.OUT, U$1.P$2
- new net EDGE_RIGHT: IC6.OUT, U$1.P$1
- new net ENCODER_LEFT_1: U$1.P$47, U$5.1
- new net ENCODER_LEFT_2: U$1.P$9, U$5.2
- new net ENCODER_RIGHT_1: U$1.P$24, U$7.1
- new net ENCODER_RIGHT_2: U$1.P$23, U$7.2
- new net IR_INT: IC2.OUT, U$1.P$20
- new net MOTOR_LEFT_1: U$1.P$44, U5.INPUT1, U5.INPUT3
- new net MOTOR_LEFT_2: U$1.P$45, U5.INPUT2, U5.INPUT4
- new net MOTOR_RIGHT_1: U$1.P$39, U2.INPUT1, U2.INPUT3
- new net MOTOR_RIGHT_2: U$1.P$67, U2.INPUT2, U2.INPUT4
- new net N$13: IC2.+IN, R35.S
- new net N$14: IC3.-IN, R15.1, U1.C
- new net N$15: IC3.+IN, R38.S
- new net N$17: R36.1, U6.A
- new net N$18: IC6.-IN, R34.1, U6.C
- new net N$19: IC6.+IN, R37.S
- new net N$3: R28.1, U1.A
- new net PI_ANALOG: R31.1, R6.1, U$1.P$38
- new net STM_RX: U$1.P$46, U$6.P$33
- new net STM_TX: U$1.P$72, U$6.P$31
- new net TAPE_LEFT: IC4.OUT, U$1.P$60
- new net TAPE_RIGHT: IC5.OUT, U$1.P$61
- net 5V_ANOLOG: now also C10.1, C11.1, C12.1, C28.1, C8.1, C9.1, IC2.V+, IC3.V+, IC4.V+, IC5.V+, IC6.V+, R34.2, R35.A, R36.2, R37.A, R38.A; no longer IC4.ON, IC5.ON
- net GND: now also C10.2, C11.2, C12.2, C28.2, C8.2, C9.2, IC2.GND, IC2.V-, IC3.GND, IC3.V-, IC6.GND, IC6.V-, R35.E, R37.E, R38.E, U$7.GND, U1.E, U1.K, U6.E, U6.K
- net IR_1: now also IC2.-IN, U$1.P$37
- net IR_2: now also U$1.P$22
- net PI_INT: now also U$1.P$19
- net SERVO_BASKET: now also U$1.P$21
- net SERVO_CLAW_1: now also U$1.P$49
- net SERVO_CLAW_2: now also U$1.P$48
Other:
- note added: "Edge Detectors"
- note added: "STM pins (pull up on IR_INT)"
- note added: "STM pins with open drain"
- note added: "STM pins with pull ups"
- note added: "STM pints with pull ups"
- note removed: "Complete: Intrrupts from GPIO and reading same singal? Comparators for ir sensors to trigger interrupts? Confirm STM pinout"
- note removed: "TODO: Assign STM pints (no pull up needed)"
- note removed: "TODO: Assign STM pints with pull ups"
- note removed: "TODO: Assign pins"
- note removed: "TODO: Assign pins on stm. Rx and tx switch."
- note removed: "TODO: Assign pins, with open drain"
- moved on the sheet: IC1G1, QSD2, R1, R15, R2, R28, R3
