File: Electrical/modules/pcb/board.sch (EAGLE design)
At the start: 108 parts, among them IC1 OP-AMP, IC2 LM311N, IC3 LM311N, IC4 LM311N, IC5 LM311N, IC6 LM311N, M1 SERVO, M2 SERVO, M3 SERVO, U1 QRD1114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

Commit message: done
Parts:
- added FUSE: 2A, SparkFun-Resistors:1KOHM-HORIZ-1/4W-5%
Connections:
- new net FUSE: C20.1, C3.1, C4.1, C7.1, FUSE.2, U$3.OUT+
- net 5V_DIGITAL: now also FUSE.1; no longer C20.1, C3.1, C4.1, C7.1, U$3.OUT+
Changed lines of the file:
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@@
 <?xml version="1.0" encoding="utf-8"?>
 <!DOCTYPE eagle SYSTEM "eagle.dtd">
-<eagle version="8.6.3">
+<eagle version="9.1.0">
 <drawing>
 <settings>
@@
 <part name="R37" library="resistor" library_urn="urn:adsk.eagle:library:348" deviceset="R-TRIMM" device="T93YA" package3d_urn="urn:adsk.eagle:package:26051/1" value="10k"/>
 <part name="R38" library="resistor" library_urn="urn:adsk.eagle:library:348" deviceset="R-TRIMM" device="T93YA" package3d_urn="urn:adsk.eagle:package:26051/1" value="10k"/>
+<part name="FUSE" library="SparkFun-Resistors" library_urn="urn:adsk.eagle:library:532" deviceset="1KOHM" device="-HORIZ-1/4W-5%" package3d_urn="urn:adsk.eagle:package:39658/1" value="2A"/>
 </parts>
 <sheets>
@@
 <instance part="R37" gate="G$1" x="350.52" y="-38.1" rot="MR180"/>
 <instance part="R38" gate="G$1" x="254" y="-40.64" rot="MR180"/>
+<instance part="FUSE" gate="G$1" x="109.22" y="129.54" rot="R180"/>
 </instances>
 <busses>
@@
 <net name="5V_DIGITAL" class="0">
 <segment>
-<pinref part="U$3" gate="G$1" pin="OUT+"/>
-<wire x1="76.2" y1="132.08" x2="81.28" y2="132.08" width="0.1524" layer="91"/>
-<label x="78.74" y="132.08" size="1.778" layer="95"/>
-<pinref part="C3" gate="G$1" pin="1"/>
-<wire x1="81.28" y1="132.08" x2="86.36" y2="132.08" width="0.1524" layer="91"/>
-<wire x1="81.28" y1="132.08" x2="81.28" y2="129.54" width="0.1524" layer="91"/>
-<wire x1="81.28" y1="129.54" x2="83.82" y2="129.54" width="0.1524" layer="91"/>
-<junction x="81.28" y="132.08"/>
-<pinref part="C4" gate="G$1" pin="1"/>
-<wire x1="83.82" y1="129.54" x2="88.9" y2="129.54" width="0.1524" layer="91"/>
-<junction x="83.82" y="129.54"/>
-<pinref part="C7" gate="G$1" pin="1"/>
-<wire x1="88.9" y1="129.54" x2="93.98" y2="129.54" width="0.1524" layer="91"/>
-<junction x="88.9" y="129.54"/>
-<pinref part="C20" gate="G$1" pin="1"/>
-<wire x1="93.98" y1="129.54" x2="99.06" y2="129.54" width="0.1524" layer="91"/>
-<junction x="93.98" y="129.54"/>
-</segment>
-<segment>
 <pinref part="U$1" gate="A" pin="P$35"/>
 <wire x1="40.64" y1="259.08" x2="45.72" y2="259.08" width="0.1524" layer="91"/>
@@
 <junction x="185.42" y="256.54"/>
 <label x="187.96" y="256.54" size="1.778" layer="95"/>
+</segment>
+<segment>
+<pinref part="FUSE" gate="G$1" pin="1"/>
+<wire x1="114.3" y1="129.54" x2="114.3" y2="139.7" width="0.1524" layer="91"/>
+<wire x1="114.3" y1="139.7" x2="111.76" y2="139.7" width="0.1524" layer="91"/>
+<label x="104.14" y="139.7" size="1.778" layer="95"/>
 </segment>
 </net>
@@
 </segment>
 </net>
+<net name="FUSE" class="0">
+<segment>
+<pinref part="C3" gate="G$1" pin="1"/>
+<wire x1="81.28" y1="129.54" x2="83.82" y2="129.54" width="0.1524" layer="91"/>
+<pinref part="C4" gate="G$1" pin="1"/>
+<wire x1="83.82" y1="129.54" x2="88.9" y2="129.54" width="0.1524" layer="91"/>
+<junction x="83.82" y="129.54"/>
+<pinref part="C7" gate="G$1" pin="1"/>
+<wire x1="88.9" y1="129.54" x2="93.98" y2="129.54" width="0.1524" layer="91"/>
+<junction x="88.9" y="129.54"/>
+<pinref part="C20" gate="G$1" pin="1"/>
+<wire x1="93.98" y1="129.54" x2="99.06" y2="129.54" width="0.1524" layer="91"/>
+<junction x="93.98" y="129.54"/>
+<pinref part="FUSE" gate="G$1" pin="2"/>
+<wire x1="99.06" y1="129.54" x2="104.14" y2="129.54" width="0.1524" layer="91"/>
+<junction x="99.06" y="129.54"/>
+<pinref part="U$3" gate="G$1" pin="OUT+"/>
+<wire x1="76.2" y1="132.08" x2="81.28" y2="132.08" width="0.1524" layer="91"/>
+<wire x1="81.28" y1="132.08" x2="81.28" y2="129.54" width="0.1524" layer="91"/>
+<label x="76.2" y="132.08" size="1.778" layer="95"/>
+</segment>
+</net>

Commit message: finalized circuit
Connections:
- new net N$32: U$1.P$105, U$1.P$106
- new net N$37: U$1.P$107, U$1.P$108
- net 5V_DIGITAL: now also U$6.P$2, U$6.P$4; no longer U$6.P$37, U$6.P$39
- net GND: now also U$6.P$14, U$6.P$20, U$6.P$25, U$6.P$30, U$6.P$34, U$6.P$39, U$6.P$6, U$6.P$9; no longer U$6.P$11, U$6.P$16, U$6.P$2, U$6.P$21, U$6.P$27, U$6.P$32, U$6.P$35, U$6.P$7
- net PI_INT: now also U$6.P$7; no longer U$6.P$4
- net R1: now also U$6.P$29; no longer U$6.P$19
- net R2: now also U$6.P$31; no longer U$6.P$23
- net R3: now also U$6.P$33; no longer U$6.P$25
- net R4: now also U$6.P$36; no longer U$6.P$26
- net R5: now also U$6.P$35; no longer U$6.P$28
- net R6: now also U$6.P$38; no longer U$6.P$30
- net R7: now also U$6.P$37; no longer U$6.P$29
- net R8: now also U$6.P$40; no longer U$6.P$34
- net STM_RX: now also U$6.P$8; no longer U$6.P$33
- net STM_TX: now also U$6.P$10; no longer U$6.P$31

Commit message: updates
Other:
- note added: "Need Pull ups"
Changed lines of the file:
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@@
 <text x="307.34" y="-10.16" size="1.778" layer="94">Edge Detectors</text>
 <text x="213.36" y="-93.98" size="1.778" layer="94">431/5 = 107 mA</text>
+<text x="182.88" y="111.76" size="1.778" layer="91">Need Pull ups</text>
 </plain>
 <instances>

Commit message: updated cube, pcb
Parts:
- removed C20, C7: 1U, capacitor-wima:C5/5
- removed FUSE: 2A, SparkFun-Resistors:1KOHM-HORIZ-1/4W-5%
- removed LIPO_B: (no value), SparkFun-Connectors:BATTERY_CONN_DEANS
- added LIPO_BIG: (no value), SparkFun-Connectors:CONN_02
- added PI_FUSE: 2A, SparkFun-Resistors:1KOHM-HORIZ-1/4W-5%
- added STM_FUSE: 300mA, SparkFun-Resistors:1KOHM-HORIZ-1/4W-5%
Connections:
- removed net FUSE: C20.1, C3.1, C4.1, C7.1, FUSE.2, U$3.OUT+
- removed net N$14: IC3.-IN, R15.1, U1.C
- removed net N$18: IC6.-IN, R34.1, U6.C
- removed net N$28: IC4.-IN, R13.1, U3.C
- removed net N$31: IC5.-IN, R16.1, U4.C
- new net +3V3: QSD1.+, QSD2.+, U$1.P$30
- new net ELA: IC3.-IN, R15.1, U$1.P$71, U1.C
- new net ERA: IC6.-IN, R34.1, U$1.P$62, U6.C
- new net PI_SUPPLY: PI_FUSE.1, U$6.P$2, U$6.P$4
- new net STM_SUPPLY: STM_FUSE.1, U$1.P$35
- new net TLA: IC4.-IN, R13.1, U$1.P$2, U3.C
- new net TRA: IC5.-IN, R16.1, U$1.P$57, U4.C
- net 5V_ANOLOG: no longer QSD1.+, QSD2.+
- net 5V_DIGITAL: now also C3.1, C4.1, PI_FUSE.2, STM_FUSE.2, U$3.OUT+; no longer FUSE.1, U$1.P$35, U$6.P$2, U$6.P$4
- net EDGE_LEFT: now also U$1.P$36; no longer U$1.P$2
- net GND: now also LIPO_BIG.1; no longer C20.2, C7.2, LIPO_B.-
- net IR_1: now also U$1.P$50; no longer U$1.P$37
- net LIPO_B_SUPPLY: now also LIPO_BIG.2; no longer LIPO_B.+
